File: kicad/MAIN/ESP32-P4-CAM-MAIN.kicad_pcb (KiCad board)
At the start: 4 copper layers, 45 x 45 mm, 128 parts, among them J1 HRO TYPE-C-31-M-12, J2 MIPI CSI 15p 1.0mm (RPi pinou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, J3 Hirose DM3AT-SF-PEJM5, J4 U.FL, J5 B2B 2x10 1.27mm (7mm mated, Q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, J7 C6/UART0 header (DNP), SW1 BOOT, SW2 RESET, SW3 USER, U1 Waveshare ESP32-P4-Module, U2 CH224A, U3 TPS259470ARPW, U4 TPS62933F, U5 TPD2E2U06DCK, U6 TPS22917DBV, U7 TPS259470ARPW (IR eFuse, DNP), U8 TPS22917DBV

Commit message: fix: route IR eFuse branch and drop CC option footprints for zero unconnected
An external review flagged the 12 DNP-only ratsnest items left after round 8.

- IR eFuse U7/R73 (still DNP) is now routed: U7.5 VBUS_SW feed from the
  In2 plane (2x 0.6/0.3 vias), U7.8 GND via, R73 moved to B under U7.
  The branch can be fitted later without bodge wires.
- CC option group R4/R5/R35/R36/C29/C30/D21/D22: a routing attempt was
  rejected by the checker (VBUS_SW plane split, GND pour fragmentation,
  ADC stubs next to CSI, 11-13 mm CC2 stubs). The symbols stay in the
  schematic as a rev B option but are excluded from the board; their
  footprints and 5 leftover CC2 stub tracks are removed.
- Pre-order gate on the master file: DRC 0 errors, 0 unconnected,
  parity 0, ERC 0; fab package, layer plots and 3D renders regenerated;
  English docs updated (round 10 in docs/90-review-log.md).

Co-Authored-By: Claude Opus 5.5 <noreply@anthropic.com>
Parts:
- removed C29, C30: 10nF DNP, Capacitor_SMD:C_0603_1608Metric
- removed D21, D22: BZT52C3V6 DNP, Diode_SMD:D_SOD-123
- removed R35, R36: 100k DNP (CC tap), Resistor_SMD:R_0603_1608Metric
- removed R4, R5: 5.1k DNP, Resistor_SMD:R_0603_1608Metric
- R73: moved to B.Cu
- moved R73 7.88 mm to (35.1, 40.9), turned to 0 degrees
Routing:
- net VBUS_SW: track 53.2 -> 62.3 mm, vias 9 -> 12
- net GND: track 324.4 -> 319.6 mm
- net CC2: track 11.7 -> 7.80 mm
- net IR_VIN_SH: track 11.6 -> 13.9 mm, vias 0 -> 2
- net IR_ILM: track 4.12 -> 5.03 mm
- net IR_SW_EN: track 45.8 -> 46.4 mm
